Commit message: cricket and fixed urdf

File: gym_cricket/assests/urdfs/cricket_robot.urdf (robot description, URDF)
Before this commit: robot cricket_robot, 42 links, 41 joints
Links:
- added link l_back_starts_track, mass 0.5; collision cylinder length=0.05 radius=0.03; visual cylinder length=0.05 radius=0.03
- added link l_front_starts_track, mass 0.5; collision cylinder length=0.05 radius=0.03; visual cylinder length=0.05 radius=0.03
- added link r_back_starts_track, mass 0.5; collision cylinder length=0.05 radius=0.03; visual cylinder length=0.05 radius=0.03
- added link r_front_starts_track, mass 0.5; collision cylinder length=0.05 radius=0.03; visual cylinder length=0.05 radius=0.03
- link l_back_jointed_track: geometry collision cylinder length=0.05 radius=0.015; visual cylinder length=0.05 radius=0.015
- link l_back_track: geometry collision box size=0.190 0.04 0.06; visual box size=0.190 0.04 0.06
- link l_front_jointed_track: geometry collision cylinder length=0.05 radius=0.015; visual cylinder length=0.05 radius=0.015
- link l_front_track: geometry collision box size=0.190 0.04 0.06; visual box size=0.190 0.04 0.06
- link r_back_jointed_track: geometry collision cylinder length=0.05 radius=0.015; visual cylinder length=0.05 radius=0.015
- link r_back_track: geometry collision box size=0.190 0.04 0.06; visual box size=0.190 0.04 0.06
- link r_front_jointed_track: geometry collision cylinder length=0.05 radius=0.015; visual cylinder length=0.05 radius=0.015
- link r_front_track: geometry collision box size=0.190 0.04 0.06; visual box size=0.190 0.04 0.06
Joints:
- added joint l_back_begin_track_joint: type continuous, parent l_back_jointed_track, child l_back_starts_track, origin xyz=0.0 0 0.0 rpy=0.0 0.0 0.0, axis 0.0 1 0.0
- added joint l_front_begin_track_joint: type continuous, parent l_front_jointed_track, child l_front_starts_track, origin xyz=0.0 0 0.0 rpy=0.0 0.0 0.0, axis 0.0 1 0.0
- added joint r_back_begin_track_joint: type continuous, parent r_back_jointed_track, child r_back_starts_track, origin xyz=0.0 0 0.0 rpy=0.0 0.0 0.0, axis 0.0 1 0.0
- added joint r_front_begin_track_joint: type continuous, parent r_front_jointed_track, child r_front_starts_track, origin xyz=0.0 0 0.0 rpy=0.0 0.0 0.0, axis 0.0 1 0.0
